File: attiny13doctor/sch/attiny13doctor.kicad_pcb (KiCad board)
At the start: 2 copper layers, 9 parts, among them J1 programmer_isp, J2 power_supply, Q1 BCR108, U1 ATMEGA8A-AU, U2 LM1117-5.0, U3 ATTINY13A-SSU

Commit message: послушал радио с двумя разными усилками и хватит
Parts:
- moved J1 5.91 mm to (270.3, 43.8)
Routing:
- net Net-(J1-Pad4): track 25.8 -> 36.5 mm
- net GND: track 65.5 -> 73.5 mm
- net +5V: track 31.8 -> 38.1 mm
- net Net-(J1-Pad6): track 11.2 -> 9.42 mm
- net Net-(J1-Pad5): track 7.86 -> 6.82 mm
